Commit message: setup initial robot parsing

File: assets/spot_simple.urdf (robot description, URDF)
Before this commit: robot spot, 15 links, 14 joints
Links:
- link body: geometry visual mesh filename=meshes/body.glb
- link fl_hip: geometry visual mesh filename=meshes/hip.glb
- link fl_lleg: geometry visual mesh filename=meshes/lleg.glb
- link fl_uleg: geometry visual mesh filename=meshes/uleg.glb
- link fr_hip: geometry visual mesh filename=meshes/hip.glb
- link fr_lleg: geometry visual mesh filename=meshes/lleg.glb
- link fr_uleg: geometry visual mesh filename=meshes/uleg.glb
- link hl_hip: geometry visual mesh filename=meshes/hip.glb
- link hl_lleg: geometry visual mesh filename=meshes/lleg.glb
- link hl_uleg: geometry visual mesh filename=meshes/uleg.glb
- link hr_hip: geometry visual mesh filename=meshes/hip.glb
- link hr_lleg: geometry visual mesh filename=meshes/lleg.glb
- link hr_uleg: geometry visual mesh filename=meshes/uleg.glb

Commit message: collisions

File: assets/spot_simple.urdf (robot description, URDF)
Before this commit: robot spot, 15 links, 14 joints
Links:
- link body: geometry visual mesh filename=meshes/visual/body.glb
- link fl_hip: geometry visual mesh filename=meshes/visual/hip.glb
- link fl_lleg: geometry collision mesh filename=meshes/collision/lleg.glb; visual mesh filename=meshes/visual/lleg.glb
- link fl_uleg: geometry visual mesh filename=meshes/visual/uleg.glb
- link fr_hip: geometry visual mesh filename=meshes/visual/hip.glb
- link fr_lleg: geometry collision mesh filename=meshes/collision/lleg.glb; visual mesh filename=meshes/visual/lleg.glb
- link fr_uleg: geometry visual mesh filename=meshes/visual/uleg.glb
- link hl_hip: geometry visual mesh filename=meshes/visual/hip.glb
- link hl_lleg: geometry collision mesh filename=meshes/collision/lleg.glb; visual mesh filename=meshes/visual/lleg.glb
- link hl_uleg: geometry visual mesh filename=meshes/visual/uleg.glb
- link hr_hip: geometry visual mesh filename=meshes/visual/hip.glb
- link hr_lleg: geometry collision mesh filename=meshes/collision/lleg.glb; visual mesh filename=meshes/visual/lleg.glb
- link hr_uleg: geometry visual mesh filename=meshes/visual/uleg.glb
